Commit message: mock

File: brazo_hardware_moveit_config/config/brazo.ros2_control.xacro (robot description, xacro)
@@ -1,5 +1,5 @@
 <?xml version="1.0"?>
 <robot xmlns:xacro="http://www.ros.org/wiki/xacro">
-  <xacro:macro name="servo_ros2_control" params="name prefix plugin">
+  <xacro:macro name="brazo_ros2_control" params="name prefix plugin">
     <ros2_control name="${name}" type="system">
       <hardware>
