Commit message: urdf y Rviz funcionó

File: brazo_hardware/description/description/urdf.xacro (robot description, xacro)
@@ -14,5 +14,5 @@
             <origin xyz="0 0 0" rpy="0 0 0" />
             <geometry>
-                <mesh filename="package://epson/meshes/base.STL" />
+                <mesh filename="package://brazo_hardware/meshes/base.STL" />
             </geometry>
             <material name="">
@@ -23,5 +23,5 @@
             <origin xyz="0 0 0" rpy="0 0 0" />
             <geometry>
-                <mesh filename="package://epson/meshes/base.STL" />
+                <mesh filename="package://brazo_hardware/meshes/base.STL" />
             </geometry>
         </collision>
@@ -41,5 +41,5 @@
             <origin xyz="0 0 0" rpy="0 0 0" />
             <geometry>
-                <mesh filename="package://epson/meshes/antebrazo.STL" />
+                <mesh filename="package://brazo_hardware/meshes/antebrazo.STL" />
             </geometry>
             <material name="">
@@ -50,5 +50,5 @@
             <origin xyz="0 0 0" rpy="0 0 0" />
             <geometry>
-                <mesh filename="package://epson/meshes/antebrazo.STL" />
+                <mesh filename="package://brazo_hardware/meshes/antebrazo.STL" />
             </geometry>
         </collision>
@@ -70,5 +70,5 @@
             <origin xyz="0 0 0" rpy="0 0 0" />
             <geometry>
-                <mesh filename="package://epson/meshes/brazo.STL" />
+                <mesh filename="package://brazo_hardware/meshes/brazo.STL" />
             </geometry>
             <material name="">
@@ -79,5 +79,5 @@
             <origin xyz="0 0 0" rpy="0 0 0" />
             <geometry>
-                <mesh filename="package://epson/meshes/brazo.STL" />
+                <mesh filename="package://brazo_hardware/meshes/brazo.STL" />
             </geometry>
         </collision>
@@ -99,5 +99,5 @@
             <origin xyz="0 0 0" rpy="0 0 0" />
             <geometry>
-                <mesh filename="package://epson/meshes/mano.STL" />
+                <mesh filename="package://brazo_hardware/meshes/mano.STL" />
             </geometry>
             <material name="">
@@ -108,5 +108,5 @@
             <origin xyz="0 0 0" rpy="0 0 0" />
             <geometry>
-                <mesh filename="package://epson/meshes/mano.STL" />
+                <mesh filename="package://brazo_hardware/meshes/mano.STL" />
             </geometry>
         </collision>
@@ -128,5 +128,5 @@
             <origin xyz="0 0 0" rpy="0 0 0" />
             <geometry>
-                <mesh filename="package://epson/meshes/dedo.STL" />
+                <mesh filename="package://brazo_hardware/meshes/dedo.STL" />
             </geometry>
             <material name="">
@@ -137,5 +137,5 @@
             <origin xyz="0 0 0" rpy="0 0 0" />
             <geometry>
-                <mesh filename="package://epson/meshes/dedo.STL" />
+                <mesh filename="package://brazo_hardware/meshes/dedo.STL" />
             </geometry>
         </collision>
@@ -189,5 +189,5 @@
     <gazebo>
         <plugin name="gazebo_ros_control" filename="libgazebo_ros_control.so">
-            <robotNamespace>/epson</robotNamespace>
+            <robotNamespace>/brazo_hardware</robotNamespace>
         </plugin>
     </gazebo>

Commit message: cambiando gazebo.py

File: brazo_hardware/description/description/urdf.xacro (robot description, xacro)
@@ -54,5 +54,6 @@
         </collision>
     </link>
-    <joint name="hombro" type="continuous">
+    <joint name="hombro" type="revolute">
+        <limit lower="-${pi/2}" upper="${pi/2}" effort="0.0" velocity="0.0"/>
         <!--<origin xyz="0 0 0.5925" rpy="0 0 0.55607" />-->
         <origin xyz="0 0 0.5925" rpy="0 0 0" />
@@ -83,5 +84,6 @@
         </collision>
     </link>
-    <joint name="codo" type="continuous">
+    <joint name="codo" type="revolute">
+        <limit lower="-${pi/2}" upper="${pi/2}" effort="0.0" velocity="0.0"/>
         <!--<origin xyz="0.4025 0 0" rpy="0 0 2.4099" /> -->
         <origin xyz="0.4025 0 0" rpy="0 0 0" />
@@ -141,5 +143,6 @@
         </collision>
     </link>
-    <joint name="muneca" type="continuous">
+    <joint name="muneca" type="revolute">
+        <limit lower="-${pi}" upper="${pi}" effort="0.0" velocity="0.0"/>
         <origin xyz="0 0 0" rpy="0 0 0" />
         <parent link="mano" />

File: brazo_hardware_moveit_config/config/brazo.ros2_control.xacro (robot description, xacro)
@@ -20,20 +20,20 @@
       </hardware>
       <joint name="${prefix}hombro">
-        <command_interface name="position"/>
+        <command_interface name="velocity"/>
         <state_interface name="position"/>
         <state_interface name="velocity"/>
       </joint>
       <joint name="${prefix}codo">
-        <command_interface name="position"/>
+        <command_interface name="velocity"/>
         <state_interface name="position"/>
         <state_interface name="velocity"/>
       </joint>
       <joint name="${prefix}articulacion">
-        <command_interface name="position"/>
+        <command_interface name="velocity"/>
         <state_interface name="position"/>
         <state_interface name="velocity"/>
       </joint>
       <joint name="${prefix}muneca">
-        <command_interface name="position"/>
+        <command_interface name="velocity"/>
         <state_interface name="position"/>
         <state_interface name="velocity"/>
