Commit message: Not moving in gazebo

File: brazo_hardware/description/description/brazo.gazebo.xacro (robot description, xacro)
@@ -2,8 +2,17 @@
 <robot>
     <!-- Gazebo Colors -->
-    <gazebo reference="motor">
-        <material>Gazebo/Blue</material>
+    <gazebo reference="base_link">
+        <material>Gazebo/Orange</material>
     </gazebo>
-    <gazebo reference="arm">
+    <gazebo reference="antebrazo">
+        <material>Gazebo/White</material>
+    </gazebo>
+    <gazebo reference="brazo">
+        <material>Gazebo/White</material>
+    </gazebo>
+    <gazebo reference="mano">
+        <material>Gazebo/White</material>
+    </gazebo>
+    <gazebo reference="dedo">
         <material>Gazebo/White</material>
     </gazebo>
@@ -13,19 +22,48 @@
             <plugin>gazebo_ros2_control/GazeboSystem</plugin>
         </hardware>
-        <joint name="servo_joint">
-            <command_interface name="position">
+        <joint name="hombro">
+            <command_interface name="velocity">
                 <param name="min">-15</param>
                 <param name="max">15</param>
             </command_interface>
             <state_interface name="position">
-                <param name="initial_value">1.0</param>
+                <param name="initial_value">0.0</param>
             </state_interface>
             <state_interface name="velocity"/>
-            <state_interface name="effort"/>
+        </joint>
+        <joint name="codo">
+            <command_interface name="velocity">
+                <param name="min">-15</param>
+                <param name="max">15</param>
+            </command_interface>
+            <state_interface name="position">
+                <param name="initial_value">0.0</param>
+            </state_interface>
+            <state_interface name="velocity"/>
+        </joint>
+        <joint name="articulacion">
+            <command_interface name="velocity">
+                <param name="min">-15</param>
+                <param name="max">15</param>
+            </command_interface>
+            <state_interface name="position">
+                <param name="initial_value">0.0</param>
+            </state_interface>
+            <state_interface name="velocity"/>
+        </joint>
+        <joint name="muneca">
+            <command_interface name="velocity">
+                <param name="min">-15</param>
+                <param name="max">15</param>
+            </command_interface>
+            <state_interface name="position">
+                <param name="initial_value">0.0</param>
+            </state_interface>
+            <state_interface name="velocity"/>
         </joint>
     </ros2_control>
     <gazebo>
         <plugin filename="libgazebo_ros2_control.so" name="gazebo_ros2_control">
-            <parameters>$(find servo_hardware)/config/servo_controllers_gazebo.yaml</parameters>
+            <parameters>$(find brazo_hardware)/config/servo_controllers_gazebo.yaml</parameters>
         </plugin>
     </gazebo>

File: brazo_hardware/description/description/brazo.simulated.xacro (robot description, xacro)
@@ -1,5 +1,5 @@
 <?xml version="1.0"?>
 <robot xmlns:xacro="http://www.ros.org/wiki/xacro" name="servo">
-    <xacro:include filename="$(find brazo_hardware)/description/description/urdf.xacro" />
-    <xacro:include filename="$(find brazo_hardware)/description/description/servo.gazebo.xacro" />
+    <xacro:include filename="$(find brazo_hardware)/description/urdf.xacro" />
+    <xacro:include filename="$(find brazo_hardware)/description/brazo.gazebo.xacro" />
 </robot>

File: brazo_hardware_moveit_config/config/brazo.ros2_control.xacro (robot description, xacro)
@@ -20,20 +20,20 @@
       </hardware>
       <joint name="${prefix}hombro">
-        <command_interface name="velocity"/>
+        <command_interface name="position"/>
         <state_interface name="position"/>
         <state_interface name="velocity"/>
       </joint>
       <joint name="${prefix}codo">
-        <command_interface name="velocity"/>
+        <command_interface name="position"/>
         <state_interface name="position"/>
         <state_interface name="velocity"/>
       </joint>
       <joint name="${prefix}articulacion">
-        <command_interface name="velocity"/>
+        <command_interface name="position"/>
         <state_interface name="position"/>
         <state_interface name="velocity"/>
       </joint>
       <joint name="${prefix}muneca">
-        <command_interface name="velocity"/>
+        <command_interface name="position"/>
         <state_interface name="position"/>
         <state_interface name="velocity"/>

File: brazo_hardware_moveit_config/config/servo.urdf.xacro (robot description, xacro)
@@ -1,8 +1,8 @@
 <?xml version="1.0"?>
-<robot xmlns:xacro="http://www.ros.org/wiki/xacro" name="servo">
+<robot xmlns:xacro="http://www.ros.org/wiki/xacro" name="epson">
     <!-- Import panda urdf file -->
-    <xacro:include filename="$(find servo_hardware)/urdf/servo.description.xacro" />
+    <xacro:include filename="$(find brazo_hardware)/description/urdf.xacro" />
     <!-- Import servo ros2_control description -->
-    <xacro:include filename="servo.ros2_control.xacro" />
+    <xacro:include filename="brazo.ros2_control.xacro" />
     <xacro:servo_ros2_control
         name="servo"

File: brazo_hardware_moveit_config/config/servo_mock.urdf.xacro (robot description, xacro)
@@ -1,4 +1,4 @@
 <?xml version="1.0"?>
-<robot xmlns:xacro="http://www.ros.org/wiki/xacro" name="servo">
+<robot xmlns:xacro="http://www.ros.org/wiki/xacro" name="epson">
     <!-- Import panda urdf file -->
     <xacro:include filename="$(find brazo_hardware)/description/urdf.xacro" />
@@ -6,5 +6,5 @@
     <xacro:include filename="brazo.ros2_control.xacro" />
     <xacro:brazo_ros2_control
-        name="servo"
+        name="brazo"
         plugin="mock_components/GenericSystem"
         prefix=""
